File: hw/rgbled.brd (EAGLE design)
At the start: 100 x 80 mm, 1 part, among them U1 ATTINY85-20P

Commit message: v1 boardu
Parts:
- added C1: (no value), resistor:C025-024X044
- added IC1: 78L05Z, linear:TO92
- added Q1, Q2, Q3: IRLZ34N, transistor-power:TO220BV
- added R1, R2, R3, R4, R5: (no value), resistor:0204/5
- added S1: (no value), switch-omron:B3F-10XX
- added X1: 22-23-2021, con-molex:22-23-2021
- added X4: (no value), con-molex:22-23-2061
- moved U1 17.0 mm to (43.2, 52.1)
Connections:
- new net +12V: IC1.3, X1.1, X4.1
- new net N$1: R5.1, S1.1, S1.2
- new net N$10: Q3.G, R4.2, U1.5
- new net N$11: Q2.G, R3.2, U1.6
- new net N$12: Q1.G, R2.2, U1.7
- new net N$2: Q1.D, X4.2
- new net N$3: Q2.D, X4.3
- new net N$4: Q3.D, X4.4
- new net N$5: R1.1, U1.2
- new net N$7: C1.1, R1.2, S1.3, S1.4, U1.3, X4.5
- net GND: now also C1.2, IC1.2, Q1.S, Q2.S, Q3.S, R2.1, R3.1, R4.1, R5.2, X1.2, X4.6
- net VCC: now also IC1.1
Routing:
- net GND: track 0.00 -> 106.7 mm
- net N$7: track 0.00 -> 58.0 mm
- net +12V: track 0.00 -> 47.0 mm
- net N$4: track 0.00 -> 21.6 mm
- net N$2: track 0.00 -> 19.0 mm
- net N$3: track 0.00 -> 15.2 mm
- net N$5: track 0.00 -> 10.2 mm
- net N$10: track 0.00 -> 3.81 mm
- net N$12: track 0.00 -> 3.81 mm
- net N$11: track 0.00 -> 3.81 mm
- net N$1: track 0.00 -> 3.38 mm
Changed lines of the file:
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@@
 </autorouter>
 <elements>
-<element name="U1" library="_hhn_attiny25_45_85" package="PDIP08_300MIL" value="ATTINY85-20P" x="50.8" y="36.83"/>
+<element name="U1" library="_hhn_attiny25_45_85" package="PDIP08_300MIL" value="ATTINY85-20P" x="43.18" y="52.07"/>
+<element name="Q1" library="transistor-power" package="TO220BV" value="IRLZ34N" x="7.62" y="50.8" rot="R270"/>
+<element name="Q2" library="transistor-power" package="TO220BV" value="IRLZ34N" x="16.51" y="50.8" rot="R270"/>
+<element name="Q3" library="transistor-power" package="TO220BV" value="IRLZ34N" x="25.4" y="50.8" rot="R270"/>
+<element name="X1" library="con-molex" package="22-23-2021" value="22-23-2021" x="45.72" y="62.23">
+<attribute name="OC_NEWARK" value="25C3832" x="45.72" y="62.23" size="1.778" layer="27" display="off"/>
+<attribute name="MPN" value="22-23-2021" x="45.72" y="62.23" size="1.778" layer="27" display="off"/>
+<attribute name="MF" value="MOLEX" x="45.72" y="62.23" size="1.778" layer="27" display="off"/>
+<attribute name="OC_FARNELL" value="1462926" x="45.72" y="62.23" size="1.778" layer="27" display="off"/>
+</element>
+<element name="X4" library="con-molex" package="22-23-2061" value="" x="11.43" y="62.23">
+<attribute name="OC_NEWARK" value="27C1933" x="11.43" y="62.23" size="1.778" layer="27" display="off"/>
+<attribute name="MPN" value="22-23-2061" x="11.43" y="62.23" size="1.778" layer="27" display="off"/>
+<attribute name="MF" value="MOLEX" x="11.43" y="62.23" size="1.778" layer="27" display="off"/>
+<attribute name="OC_FARNELL" value="1462922" x="11.43" y="62.23" size="1.778" layer="27" display="off"/>
+</element>
+<element name="IC1" library="linear" package="TO92" value="78L05Z" x="39.37" y="62.23" rot="R90"/>
+<element name="R1" library="resistor" package="0204/5" value="" x="34.29" y="50.8" rot="R90"/>
+<element name="C1" library="resistor" package="C025-024X044" value="" x="30.48" y="49.53" rot="R270"/>
+<element name="R2" library="resistor" package="0204/5" value="" x="8.89" y="50.8" rot="R90"/>
+<element name="R3" library="resistor" package="0204/5" value="" x="17.78" y="50.8" rot="R90"/>
+<element name="R4" library="resistor" package="0204/5" value="" x="26.67" y="50.8" rot="R90"/>
+<element name="S1" library="switch-omron" package="B3F-10XX" value="" x="26.67" y="60.96" rot="R180">
+<attribute name="OC_NEWARK" value="36M3542" x="26.67" y="60.96" size="1.778" layer="27" rot="R180" display="off"/>
+<attribute name="MPN" value="B3F-1000" x="26.67" y="60.96" size="1.778" layer="27" rot="R180" display="off"/>
+<attribute name="MF" value="" x="26.67" y="60.96" size="1.778" layer="27" rot="R180" display="off"/>
+<attribute name="OC_FARNELL" value="176432" x="26.67" y="60.96" size="1.778" layer="27" rot="R180" display="off"/>
+</element>
+<element name="R5" library="resistor" package="0204/5" value="" x="35.56" y="58.42"/>
 </elements>
 <signals>
 <signal name="VCC">
 <contactref element="U1" pad="8"/>
+<contactref element="IC1" pad="1"/>
+<contactref element="U1" pad="8"/>
+<wire x1="39.37" y1="60.96" x2="39.37" y2="55.88" width="0" layer="19" extent="1-1"/>
 </signal>
 <signal name="GND">
 <contactref element="U1" pad="4"/>
+<contactref element="X1" pad="2"/>
+<contactref element="U1" pad="4"/>
+<contactref element="IC1" pad="2"/>
+<contactref element="Q1" pad="S"/>
+<contactref element="Q2" pad="S"/>
+<contactref element="Q3" pad="S"/>
+<contactref element="X4" pad="6"/>
+<contactref element="C1" pad="2"/>
+<contactref element="R2" pad="1"/>
+<contactref element="R3" pad="1"/>
+<contactref element="R4" pad="1"/>
+<contactref element="R5" pad="2"/>
+<wire x1="5.08" y1="48.26" x2="8.89" y2="48.26" width="0.4064" layer="16"/>
+<wire x1="8.89" y1="48.26" x2="13.97" y2="48.26" width="0.4064" layer="16"/>
+<wire x1="13.97" y1="48.26" x2="17.78" y2="48.26" width="0.4064" layer="16"/>
+<wire x1="17.78" y1="48.26" x2="22.86" y2="48.26" width="0.4064" layer="16"/>
+<wire x1="22.86" y1="48.26" x2="26.67" y2="48.26" width="0.4064" layer="16"/>
+<wire x1="26.67" y1="48.26" x2="30.48" y2="48.26" width="0.4064" layer="16"/>
+<wire x1="30.48" y1="48.26" x2="30.48" y2="45.72" width="0.4064" layer="16"/>
+<wire x1="30.48" y1="45.72" x2="46.99" y2="45.72" width="0.4064" layer="16"/>
+<wire x1="46.99" y1="45.72" x2="46.99" y2="48.26" width="0.4064" layer="16"/>
+<wire x1="46.99" y1="62.23" x2="50.8" y2="62.23" width="0.4064" layer="16"/>
+<wire x1="50.8" y1="62.23" x2="50.8" y2="48.26" width="0.4064" layer="16"/>
+<wire x1="50.8" y1="48.26" x2="46.99" y2="48.26" width="0.4064" layer="16"/>
+<wire x1="38.1" y1="58.42" x2="46.99" y2="58.42" width="0.4064" layer="16"/>
+<wire x1="46.99" y1="58.42" x2="46.99" y2="62.23" width="0.4064" layer="16"/>
+<wire x1="17.78" y1="62.23" x2="17.78" y2="60.96" width="0.4064" layer="16"/>
+<wire x1="38.1" y1="58.42" x2="37.465" y2="58.42" width="0.4064" layer="16"/>
+<wire x1="37.465" y1="58.42" x2="37.465" y2="60.96" width="0.4064" layer="16"/>
+<wire x1="37.465" y1="60.96" x2="37.465" y2="62.23" width="0.4064" layer="16"/>
+<wire x1="17.78" y1="60.96" x2="37.465" y2="60.96" width="0.4064" layer="16"/>
+</signal>
+<signal name="+12V">
+<contactref element="X1" pad="1"/>
+<contactref element="IC1" pad="3"/>
+<contactref element="X4" pad="1"/>
+<wire x1="5.08" y1="62.23" x2="5.08" y2="66.04" width="0.4064" layer="16"/>
+<wire x1="5.08" y1="66.04" x2="39.37" y2="66.04" width="0.4064" layer="16"/>
+<wire x1="39.37" y1="66.04" x2="39.37" y2="63.5" width="0.4064" layer="16"/>
+<wire x1="39.37" y1="63.5" x2="44.45" y2="63.5" width="0.4064" layer="16"/>
+<wire x1="44.45" y1="63.5" x2="44.45" y2="62.23" width="0.4064" layer="16"/>
+</signal>
+<signal name="N$2">
+<contactref element="X4" pad="2"/>
+<contactref element="Q1" pad="D"/>
+<wire x1="5.08" y1="50.8" x2="2.54" y2="50.8" width="0.4064" layer="16"/>
+<wire x1="2.54" y1="50.8" x2="2.54" y2="57.15" width="0.4064" layer="16"/>
+<wire x1="2.54" y1="57.15" x2="7.62" y2="57.15" width="0.4064" layer="16"/>
+<wire x1="7.62" y1="57.15" x2="7.62" y2="62.23" width="0.4064" layer="16"/>
+</signal>
+<signal name="N$3">
+<contactref element="X4" pad="3"/>
+<contactref element="Q2" pad="D"/>
+<wire x1="13.97" y1="50.8" x2="11.43" y2="50.8" width="0.4064" layer="16"/>
+<wire x1="11.43" y1="50.8" x2="11.43" y2="57.15" width="0.4064" layer="16"/>
+<wire x1="11.43" y1="57.15" x2="10.16" y2="57.15" width="0.4064" layer="16"/>
+<wire x1="10.16" y1="57.15" x2="10.16" y2="62.23" width="0.4064" layer="16"/>
+</signal>
+<signal name="N$4">
+<contactref element="X4" pad="4"/>
+<contactref element="Q3" pad="D"/>
+<wire x1="22.86" y1="50.8" x2="20.32" y2="50.8" width="0.4064" layer="16"/>
+<wire x1="20.32" y1="50.8" x2="20.32" y2="57.15" width="0.4064" layer="16"/>
+<wire x1="20.32" y1="57.15" x2="12.7" y2="57.15" width="0.4064" layer="16"/>
+<wire x1="12.7" y1="57.15" x2="12.7" y2="62.23" width="0.4064" layer="16"/>
+</signal>
+<signal name="N$5">
+<contactref element="U1" pad="2"/>
+<contactref element="R1" pad="1"/>
+<wire x1="34.29" y1="48.26" x2="34.29" y2="49.53" width="0.4064" layer="16"/>
+<wire x1="34.29" y1="49.53" x2="41.91" y2="49.53" width="0.4064" layer="16"/>
+<wire x1="41.91" y1="49.53" x2="41.91" y2="48.26" width="0.4064" layer="16"/>
+</signal>
+<signal name="N$10">
+<contactref element="Q3" pad="G"/>
+<contactref element="R4" pad="2"/>
+<contactref element="U1" pad="5"/>
+<wire x1="22.86" y1="53.34" x2="46.99" y2="55.88" width="0" layer="19" extent="1-1"/>
+<wire x1="22.86" y1="53.34" x2="26.67" y2="53.34" width="0.4064" layer="16"/>
+</signal>
+<signal name="N$11">
+<contactref element="Q2" pad="G"/>
+<contactref element="R3" pad="2"/>
+<contactref element="U1" pad="6"/>
+<wire x1="13.97" y1="53.34" x2="44.45" y2="55.88" width="0" layer="19" extent="1-1"/>
+<wire x1="13.97" y1="53.34" x2="17.78" y2="53.34" width="0.4064" layer="16"/>
+</signal>
+<signal name="N$12">
+<contactref element="Q1" pad="G"/>
+<contactref element="R2" pad="2"/>
+<contactref element="U1" pad="7"/>
+<wire x1="5.08" y1="53.34" x2="8.89" y2="53.34" width="0.4064" layer="16"/>
+<wire x1="8.89" y1="53.34" x2="41.91" y2="55.88" width="0" layer="19" extent="1-1"/>
+</signal>
+<signal name="N$7">
+<contactref element="R1" pad="2"/>
+<contactref element="C1" pad="1"/>
+<contactref element="X4" pad="5"/>
+<contactref element="U1" pad="3"/>
+<contactref element="S1" pad="3"/>
+<contactref element="S1" pad="4"/>
+<wire x1="23.4188" y1="63.2206" x2="29.9212" y2="63.2206" width="0" layer="19" extent="1-1"/>
+<wire x1="15.24" y1="62.23" x2="15.24" y2="63.5" width="0.4064" layer="16"/>
+<wire x1="15.24" y1="63.5" x2="23.4188" y2="63.5" width="0.4064" layer="16"/>
+<wire x1="23.4188" y1="63.5" x2="23.4188" y2="63.2206" width="0.4064" layer="16"/>
+<wire x1="15.24" y1="62.23" x2="15.24" y2="58.42" width="0.4064" layer="16"/>
+<wire x1="15.24" y1="58.42" x2="21.59" y2="58.42" width="0.4064" layer="16"/>
+<wire x1="21.59" y1="58.42" x2="21.59" y2="57.15" width="0.4064" layer="16"/>
+<wire x1="21.59" y1="57.15" x2="30.48" y2="57.15" width="0.4064" layer="16"/>
+<wire x1="30.48" y1="57.15" x2="30.48" y2="50.8" width="0.4064" layer="16"/>
+<wire x1="44.45" y1="48.26" x2="44.45" y2="50.8" width="0.4064" layer="16"/>
+<wire x1="44.45" y1="50.8" x2="34.29" y2="50.8" width="0.4064" layer="16"/>
+<wire x1="34.29" y1="50.8" x2="34.29" y2="53.34" width="0.4064" layer="16"/>
+<wire x1="34.29" y1="53.34" x2="30.48" y2="53.34" width="0.4064" layer="16"/>
+<wire x1="30.48" y1="53.34" x2="30.48" y2="50.8" width="0.4064" layer="16"/>
+</signal>
+<signal name="N$1">
+<contactref element="S1" pad="1"/>
+<contactref element="R5" pad="1"/>
+<contactref element="S1" pad="2"/>
+<wire x1="23.4188" y1="58.6994" x2="29.9212" y2="58.6994" width="0" layer="19" extent="1-1"/>
+<wire x1="29.9212" y1="58.6994" x2="33.02" y2="58.6994" width="0.4064" layer="16"/>
+<wire x1="33.02" y1="58.6994" x2="33.02" y2="58.42" width="0.4064" layer="16"/>
 </signal>
 </signals>

Commit message: upravy sch
Parts:
- C1: value (none) -> 100p
- IC1: value 78L05Z -> LE33CZ
- R1: value (none) -> 10M
- R2, R3, R4, R5: value (none) -> 10K
Changed lines of the file:
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@@
 <attribute name="OC_FARNELL" value="1462922" x="11.43" y="62.23" size="1.778" layer="27" display="off"/>
 </element>
-<element name="IC1" library="linear" package="TO92" value="78L05Z" x="39.37" y="62.23" rot="R90"/>
-<element name="R1" library="resistor" package="0204/5" value="" x="34.29" y="50.8" rot="R90"/>
-<element name="C1" library="resistor" package="C025-024X044" value="" x="30.48" y="49.53" rot="R270"/>
-<element name="R2" library="resistor" package="0204/5" value="" x="8.89" y="50.8" rot="R90"/>
-<element name="R3" library="resistor" package="0204/5" value="" x="17.78" y="50.8" rot="R90"/>
-<element name="R4" library="resistor" package="0204/5" value="" x="26.67" y="50.8" rot="R90"/>
+<element name="IC1" library="linear" package="TO92" value="LE33CZ" x="39.37" y="62.23" rot="R90"/>
+<element name="R1" library="resistor" package="0204/5" value="10M" x="34.29" y="50.8" rot="R90"/>
+<element name="C1" library="resistor" package="C025-024X044" value="100p" x="30.48" y="49.53" rot="R270"/>
+<element name="R2" library="resistor" package="0204/5" value="10K" x="8.89" y="50.8" rot="R90"/>
+<element name="R3" library="resistor" package="0204/5" value="10K" x="17.78" y="50.8" rot="R90"/>
+<element name="R4" library="resistor" package="0204/5" value="10K" x="26.67" y="50.8" rot="R90"/>
 <element name="S1" library="switch-omron" package="B3F-10XX" value="" x="26.67" y="60.96" rot="R180">
 <attribute name="OC_NEWARK" value="36M3542" x="26.67" y="60.96" size="1.778" layer="27" rot="R180" display="off"/>
@@
 <attribute name="OC_FARNELL" value="176432" x="26.67" y="60.96" size="1.778" layer="27" rot="R180" display="off"/>
 </element>
-<element name="R5" library="resistor" package="0204/5" value="" x="35.56" y="58.42"/>
+<element name="R5" library="resistor" package="0204/5" value="10K" x="35.56" y="58.42"/>
 </elements>
 <signals>

Commit message: upravy problikavani
Parts:
- added R6, R7, R8: 1K, resistor:0204/5
- R2, R3, R4: value 10K -> 1M
Connections:
- new net N$6: Q1.G, R2.2, R6.1
- new net N$8: Q2.G, R3.2, R7.1
- new net N$9: Q3.G, R4.2, R8.1
- net N$10: now also R8.2; no longer Q3.G, R4.2
- net N$11: now also R7.2; no longer Q2.G, R3.2
- net N$12: now also R6.2; no longer Q1.G, R2.2
Routing:
- net N$12: track 3.81 -> 39.4 mm
- net N$11: track 3.81 -> 33.0 mm
- net N$10: track 3.81 -> 26.7 mm
- net N$9: track 0.00 -> 6.35 mm
- net N$8: track 0.00 -> 6.35 mm
- net N$6: track 0.00 -> 6.35 mm
- net VCC: track 0.00 -> 5.08 mm
Changed lines of the file:
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@@
 <element name="R1" library="resistor" package="0204/5" value="10M" x="34.29" y="50.8" rot="R90"/>
 <element name="C1" library="resistor" package="C025-024X044" value="100p" x="30.48" y="49.53" rot="R270"/>
-<element name="R2" library="resistor" package="0204/5" value="10K" x="8.89" y="50.8" rot="R90"/>
-<element name="R3" library="resistor" package="0204/5" value="10K" x="17.78" y="50.8" rot="R90"/>
-<element name="R4" library="resistor" package="0204/5" value="10K" x="26.67" y="50.8" rot="R90"/>
+<element name="R2" library="resistor" package="0204/5" value="1M" x="8.89" y="50.8" rot="R90"/>
+<element name="R3" library="resistor" package="0204/5" value="1M" x="17.78" y="50.8" rot="R90"/>
+<element name="R4" library="resistor" package="0204/5" value="1M" x="26.67" y="50.8" rot="R90"/>
 <element name="S1" library="switch-omron" package="B3F-10XX" value="" x="26.67" y="60.96" rot="R180">
 <attribute name="OC_NEWARK" value="36M3542" x="26.67" y="60.96" size="1.778" layer="27" rot="R180" display="off"/>
@@
 </element>
 <element name="R5" library="resistor" package="0204/5" value="10K" x="35.56" y="58.42"/>
+<element name="R6" library="resistor" package="0204/5" value="1K" x="7.62" y="55.88"/>
+<element name="R7" library="resistor" package="0204/5" value="1K" x="16.51" y="55.88"/>
+<element name="R8" library="resistor" package="0204/5" value="1K" x="25.4" y="55.88"/>
 </elements>
 <signals>
@@
 <contactref element="IC1" pad="1"/>
 <contactref element="U1" pad="8"/>
-<wire x1="39.37" y1="60.96" x2="39.37" y2="55.88" width="0" layer="19" extent="1-1"/>
+<wire x1="39.37" y1="60.96" x2="39.37" y2="55.88" width="0.4064" layer="1"/>
 </signal>
 <signal name="GND">
@@
 </signal>
 <signal name="N$10">
-<contactref element="Q3" pad="G"/>
-<contactref element="R4" pad="2"/>
 <contactref element="U1" pad="5"/>
-<wire x1="22.86" y1="53.34" x2="46.99" y2="55.88" width="0" layer="19" extent="1-1"/>
-<wire x1="22.86" y1="53.34" x2="26.67" y2="53.34" width="0.4064" layer="16"/>
+<contactref element="R8" pad="2"/>
+<wire x1="46.99" y1="55.88" x2="46.99" y2="52.07" width="0.4064" layer="1"/>
+<wire x1="46.99" y1="52.07" x2="27.94" y2="52.07" width="0.4064" layer="1"/>
+<wire x1="27.94" y1="52.07" x2="27.94" y2="55.88" width="0.4064" layer="1"/>
 </signal>
 <signal name="N$11">
-<contactref element="Q2" pad="G"/>
-<contactref element="R3" pad="2"/>
 <contactref element="U1" pad="6"/>
-<wire x1="13.97" y1="53.34" x2="44.45" y2="55.88" width="0" layer="19" extent="1-1"/>
-<wire x1="13.97" y1="53.34" x2="17.78" y2="53.34" width="0.4064" layer="16"/>
+<contactref element="R7" pad="2"/>
+<wire x1="44.45" y1="55.88" x2="44.45" y2="53.34" width="0.4064" layer="1"/>
+<wire x1="44.45" y1="53.34" x2="31.75" y2="53.34" width="0.4064" layer="1"/>
+<wire x1="31.75" y1="53.34" x2="31.75" y2="57.15" width="0.4064" layer="1"/>
+<wire x1="31.75" y1="57.15" x2="19.05" y2="57.15" width="0.4064" layer="1"/>
+<wire x1="19.05" y1="57.15" x2="19.05" y2="55.88" width="0.4064" layer="1"/>
 </signal>
 <signal name="N$12">
-<contactref element="Q1" pad="G"/>
-<contactref element="R2" pad="2"/>
 <contactref element="U1" pad="7"/>
-<wire x1="5.08" y1="53.34" x2="8.89" y2="53.34" width="0.4064" layer="16"/>
-<wire x1="8.89" y1="53.34" x2="41.91" y2="55.88" width="0" layer="19" extent="1-1"/>
+<contactref element="R6" pad="2"/>
+<wire x1="41.91" y1="55.88" x2="41.91" y2="54.61" width="0.4064" layer="1"/>
+<wire x1="41.91" y1="54.61" x2="34.29" y2="54.61" width="0.4064" layer="1"/>
+<wire x1="34.29" y1="54.61" x2="34.29" y2="58.42" width="0.4064" layer="1"/>
+<wire x1="34.29" y1="58.42" x2="10.16" y2="58.42" width="0.4064" layer="1"/>
+<wire x1="10.16" y1="58.42" x2="10.16" y2="55.88" width="0.4064" layer="1"/>
 </signal>
 <signal name="N$7">
@@
 <wire x1="33.02" y1="58.6994" x2="33.02" y2="58.42" width="0.4064" layer="16"/>
 </signal>
+<signal name="N$8">
+<contactref element="Q2" pad="G"/>
+<contactref element="R3" pad="2"/>
+<wire x1="13.97" y1="53.34" x2="17.78" y2="53.34" width="0.4064" layer="16"/>
+<contactref element="R7" pad="1"/>
+<wire x1="13.97" y1="55.88" x2="13.97" y2="53.34" width="0.4064" layer="16"/>
+</signal>
+<signal name="N$9">
+<contactref element="Q3" pad="G"/>
+<contactref element="R4" pad="2"/>
+<wire x1="22.86" y1="53.34" x2="26.67" y2="53.34" width="0.4064" layer="16"/>
+<contactref element="R8" pad="1"/>
+<wire x1="22.86" y1="55.88" x2="22.86" y2="53.34" width="0.4064" layer="16"/>
+</signal>
+<signal name="N$6">
+<contactref element="Q1" pad="G"/>
+<contactref element="R2" pad="2"/>
+<contactref element="R6" pad="1"/>
+<wire x1="5.08" y1="55.88" x2="5.08" y2="53.34" width="0.4064" layer="16"/>
+<wire x1="5.08" y1="53.34" x2="8.89" y2="53.34" width="0.4064" layer="16"/>
+</signal>
 </signals>
